File: hw/v0p1/RPi_Connector.sch (KiCad schematic (older format))
At the start: 1 part, among them P1 Conn_02x20_Odd_Even

Commit message: Updated BOM
Parts:
- P1: LCSC (none) -> C50982
Changed lines of the file:
@@
 F 2 "Connector_PinSocket_2.54mm:PinSocket_2x20_P2.54mm_Vertical" H -2000 1350 50  0001 C CNN
 F 3 "" H -2000 1350 50  0001 C CNN
+F 4 "C50982" H 2850 2300 50  0001 C CNN "LCSC"
 	1    2850 2300
 	1    0    0    -1
