File: hw/v0p1/FTDI_Controller.sch (KiCad schematic (older format))
At the start: 12 parts, among them J4 USB_B_Micro, J5 Conn_01x06, U2 FT230XS

Commit message: Updated BOM
Parts:
- J4: LCSC (none) -> C319170
- U2: LCSC (none) -> C69082
Changed lines of the file:
@@
 F 2 "Package_SO:SSOP-16_3.9x4.9mm_P0.635mm" H 6900 2300 50  0001 C CNN
 F 3 "http://www.ftdichip.com/Products/ICs/FT230X.html" H 6450 2950 50  0001 C CNN
+F 4 "C69082" H 6450 2950 50  0001 C CNN "LCSC"
 	1    6450 2950
 	1    0    0    -1
@@
 F 2 "Connector_USB:USB_Micro-B_Wuerth_629105150521" H 4450 2150 50  0001 C CNN
 F 3 "~" H 4450 2150 50  0001 C CNN
+F 4 "C319170" H 4300 2200 50  0001 C CNN "LCSC"
 	1    4300 2200
 	1    0    0    -1

Commit message: Updated
Connections:
- net labels added: USB_DM, USB_DP
- wire segments 50 -> 45
Other:
- moved on the sheet: C3, C4, C5
Changed lines of the file:
@@
 L Device:C_Small C3
 U 1 1 5F638CAF
-P 4800 2350
-F 0 "C3" H 4892 2396 50  0000 L CNN
-F 1 "47pF" H 4892 2305 50  0000 L CNN
-F 2 "Capacitor_SMD:C_0805_2012Metric" H 4800 2350 50  0001 C CNN
-F 3 "~" H 4800 2350 50  0001 C CNN
-F 4 "C123648" H 4800 2350 50  0001 C CNN "LCSC"
-	1    4800 2350
-	1    0    0    -1
+P 5000 2750
+F 0 "C3" H 4800 2750 50  0000 L CNN
+F 1 "47pF" H 4750 2650 50  0000 L CNN
+F 2 "Capacitor_SMD:C_0805_2012Metric" H 5000 2750 50  0001 C CNN
+F 3 "~" H 5000 2750 50  0001 C CNN
+F 4 "C123648" H 5000 2750 50  0001 C CNN "LCSC"
+	1    5000 2750
+	-1   0    0    1
 $EndComp
 $Comp
 L Device:C_Small C4
 U 1 1 5F63A5A8
-P 4800 2800
-F 0 "C4" H 4892 2846 50  0000 L CNN
-F 1 "47pF" H 4892 2755 50  0000 L CNN
-F 2 "Capacitor_SMD:C_0805_2012Metric" H 4800 2800 50  0001 C CNN
-F 3 "~" H 4800 2800 50  0001 C CNN
-F 4 "C123648" H 4800 2800 50  0001 C CNN "LCSC"
-	1    4800 2800
-	1    0    0    -1
-$EndComp
-Wire Wire Line
-	4600 2200 4800 2200
-Wire Wire Line
-	4800 2200 4800 2250
-Wire Wire Line
-	5150 2200 5150 2850
-Wire Wire Line
-	5150 2850 5450 2850
-Wire Wire Line
-	4800 2200 5150 2200
-Connection ~ 4800 2200
-Wire Wire Line
-	4600 2300 4650 2300
-Wire Wire Line
-	4650 2700 4800 2700
-Wire Wire Line
-	4800 2700 5100 2700
-Wire Wire Line
-	5100 2950 5450 2950
+P 5000 3050
+F 0 "C4" H 5092 3096 50  0000 L CNN
+F 1 "47pF" H 5092 3005 50  0000 L CNN
+F 2 "Capacitor_SMD:C_0805_2012Metric" H 5000 3050 50  0001 C CNN
+F 3 "~" H 5000 3050 50  0001 C CNN
+F 4 "C123648" H 5000 3050 50  0001 C CNN "LCSC"
+	1    5000 3050
+	1    0    0    -1
+$EndComp
 $Comp
 L power:GND #PWR028
 U 1 1 5F63EB83
-P 4800 2450
-F 0 "#PWR028" H 4800 2200 50  0001 C CNN
-F 1 "GND" H 4805 2277 50  0000 C CNN
-F 2 "" H 4800 2450 50  0001 C CNN
-F 3 "" H 4800 2450 50  0001 C CNN
-	1    4800 2450
-	1    0    0    -1
+P 5000 2650
+F 0 "#PWR028" H 5000 2400 50  0001 C CNN
+F 1 "GND" H 5005 2477 50  0000 C CNN
+F 2 "" H 5000 2650 50  0001 C CNN
+F 3 "" H 5000 2650 50  0001 C CNN
+	1    5000 2650
+	-1   0    0    1
 $EndComp
 $Comp
 L power:GND #PWR029
 U 1 1 5F63F10D
-P 4800 2900
-F 0 "#PWR029" H 4800 2650 50  0001 C CNN
-F 1 "GND" H 4805 2727 50  0000 C CNN
-F 2 "" H 4800 2900 50  0001 C CNN
-F 3 "" H 4800 2900 50  0001 C CNN
-	1    4800 2900
-	1    0    0    -1
-$EndComp
-Wire Wire Line
-	5100 2700 5100 2950
-Connection ~ 4800 2700
-Wire Wire Line
-	4650 2300 4650 2700
+P 5000 3150
+F 0 "#PWR029" H 5000 2900 50  0001 C CNN
+F 1 "GND" H 5005 2977 50  0000 C CNN
+F 2 "" H 5000 3150 50  0001 C CNN
+F 3 "" H 5000 3150 50  0001 C CNN
+	1    5000 3150
+	1    0    0    -1
+$EndComp
+Connection ~ 5000 2950
 $Comp
 L Device:C_Small C5
 U 1 1 5F640973
-P 5200 3850
-F 0 "C5" H 5292 3896 50  0000 L CNN
-F 1 "100nF" H 5292 3805 50  0000 L CNN
-F 2 "Capacitor_SMD:C_0805_2012Metric" H 5200 3850 50  0001 C CNN
-F 3 "~" H 5200 3850 50  0001 C CNN
-F 4 "C83055" H 5200 3850 50  0001 C CNN "LCSC"
-	1    5200 3850
-	1    0    0    -1
-$EndComp
-Text Label 4650 3450 0    50   ~ 0
+P 7600 4350
+F 0 "C5" H 7692 4396 50  0000 L CNN
+F 1 "100nF" H 7692 4305 50  0000 L CNN
+F 2 "Capacitor_SMD:C_0805_2012Metric" H 7600 4350 50  0001 C CNN
+F 3 "~" H 7600 4350 50  0001 C CNN
+F 4 "C83055" H 7600 4350 50  0001 C CNN "LCSC"
+	1    7600 4350
+	1    0    0    -1
+$EndComp
+Text Label 7050 3950 0    50   ~ 0
 FTDI_RESET
 Wire Wire Line
-	4650 3450 5200 3450
-Text Label 4650 3550 0    50   ~ 0
+	7050 3950 7600 3950
+Text Label 7050 4050 0    50   ~ 0
 FTDI_3v3_Out
 Wire Wire Line
-	4650 3550 5200 3550
-Text Label 4650 3650 0    50   ~ 0
+	7050 4050 7600 4050
+Text Label 7050 4150 0    50   ~ 0
 FTDI_VCCIO
 Wire Wire Line
-	4650 3650 5200 3650
+	7050 4150 7600 4150
 $Comp
 L power:GND #PWR030
 U 1 1 5F64542D
-P 5200 4050
-F 0 "#PWR030" H 5200 3800 50  0001 C CNN
-F 1 "GND" H 5205 3877 50  0000 C CNN
-F 2 "" H 5200 4050 50  0001 C CNN
-F 3 "" H 5200 4050 50  0001 C CNN
-	1    5200 4050
-	1    0    0    -1
-$EndComp
-Wire Wire Line
-	5200 3450 5200 3550
-Connection ~ 5200 3550
-Wire Wire Line
-	5200 3550 5200 3650
-Connection ~ 5200 3650
-Wire Wire Line
-	5200 3650 5200 3750
-Wire Wire Line
-	5200 3950 5200 4050
+P 7600 4550
+F 0 "#PWR030" H 7600 4300 50  0001 C CNN
+F 1 "GND" H 7605 4377 50  0000 C CNN
+F 2 "" H 7600 4550 50  0001 C CNN
+F 3 "" H 7600 4550 50  0001 C CNN
+	1    7600 4550
+	1    0    0    -1
+$EndComp
+Wire Wire Line
+	7600 3950 7600 4050
+Connection ~ 7600 4050
+Wire Wire Line
+	7600 4050 7600 4150
+Connection ~ 7600 4150
+Wire Wire Line
+	7600 4150 7600 4250
+Wire Wire Line
+	7600 4450 7600 4550
 Wire Wire Line
 	3800 3550 4000 3550
@@
 Text Label 7200 2850 0    50   ~ 0
 FTDI_CTS
+Text Label 4650 2850 0    50   ~ 0
+USB_DM
+Text Label 4650 2950 0    50   ~ 0
+USB_DP
+Wire Wire Line
+	5000 2950 5450 2950
+Wire Wire Line
+	4650 2850 5000 2850
+Connection ~ 5000 2850
+Wire Wire Line
+	4650 2950 5000 2950
+Wire Wire Line
+	5000 2850 5450 2850
+Text Label 4650 2300 0    50   ~ 0
+USB_DM
+Text Label 4650 2200 0    50   ~ 0
+USB_DP
+Wire Wire Line
+	4600 2300 4950 2300
+Wire Wire Line
+	4600 2200 4950 2200
 $EndSCHEMATC
