File: hw/v0p1/NetworkBreaker.kicad_pcb (KiCad board)
At the start: 2 copper layers, 65 x 56 mm, 45 parts, among them J1 8P8C_Shielded, J2 8P8C_Shielded, J3 8P8C_Shielded, J4 USB_B_Micro, J5 Conn_01x06, K1 M4-5HAW, K2 M4-5HAW, K3 M4-5HAW, K4 M4-5HAW, P1 Conn_02x20_Odd_Even, Q1 2N3904, Q2 2N3904, Q3 2N3904, Q4 2N3904, U1 TLP627-4, U2 FT230XS

Commit message: Updated part LCSC part numbers
Parts:
- D1, D2, D3, D4: value LED_Small -> Green
- R1, R2, R3, R4: value R_Small -> 220
- R5, R6, R7, R8: value R_Small -> 10k
Changed lines of the file:
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@@
     (add_net /FTDI_Controller/FTDI_RXD)
     (add_net /FTDI_Controller/FTDI_TXD)
+    (add_net "/RPi_Connector/GPIO10(SPI0_MOSI)")
+    (add_net "/RPi_Connector/GPIO11(SPI0_SCK)")
+    (add_net "/RPi_Connector/GPIO12(PWM0)")
+    (add_net "/RPi_Connector/GPIO14(TXD0)")
+    (add_net "/RPi_Connector/GPIO15(RXD0)")
+    (add_net /RPi_Connector/GPIO16)
+    (add_net "/RPi_Connector/GPIO17(GEN0)")
+    (add_net "/RPi_Connector/GPIO18(GEN1)(PWM0)")
+    (add_net "/RPi_Connector/GPIO2(SDA1)")
+    (add_net "/RPi_Connector/GPIO20(SPI1_MOSI)")
+    (add_net "/RPi_Connector/GPIO21(SPI1_SCK)")
+    (add_net "/RPi_Connector/GPIO22(GEN3)")
+    (add_net "/RPi_Connector/GPIO23(GEN4)")
+    (add_net "/RPi_Connector/GPIO24(GEN5)")
+    (add_net "/RPi_Connector/GPIO25(GEN6)")
+    (add_net /RPi_Connector/GPIO26)
+    (add_net "/RPi_Connector/GPIO27(GEN2)")
+    (add_net "/RPi_Connector/GPIO3(SCL1)")
+    (add_net "/RPi_Connector/GPIO4(GCLK)")
+    (add_net "/RPi_Connector/GPIO7(SPI1_CE_N)")
+    (add_net "/RPi_Connector/GPIO8(SPI0_CE_N)")
+    (add_net "/RPi_Connector/GPIO9(SPI0_MISO)")
+    (add_net /RPi_Connector/ID_SC)
+    (add_net /RPi_Connector/ID_SD)
     (add_net GND)
     (add_net GPIO13)
@@
     (add_net "Net-(D7-Pad2)")
     (add_net "Net-(D8-Pad2)")
+    (add_net "Net-(J4-Pad4)")
     (add_net "Net-(Q1-Pad2)")
     (add_net "Net-(Q2-Pad2)")
@@
       (effects (font (size 1 1) (thickness 0.15)) (justify mirror))
     )
-    (fp_text value R_Small (at 0 -1.65 90) (layer B.Fab)
+    (fp_text value 10k (at 0 -1.65 90) (layer B.Fab)
       (effects (font (size 1 1) (thickness 0.15)) (justify mirror))
     )
@@
       (effects (font (size 1 1) (thickness 0.15)) (justify mirror))
     )
-    (fp_text value R_Small (at 0 -1.65 90) (layer B.Fab)
+    (fp_text value 10k (at 0 -1.65 90) (layer B.Fab)
       (effects (font (size 1 1) (thickness 0.15)) (justify mirror))
     )
@@
       (effects (font (size 1 1) (thickness 0.15)) (justify mirror))
     )
-    (fp_text value R_Small (at 0 -1.65 90) (layer B.Fab)
+    (fp_text value 10k (at 0 -1.65 90) (layer B.Fab)
       (effects (font (size 1 1) (thickness 0.15)) (justify mirror))
     )
@@
       (effects (font (size 1 1) (thickness 0.15)) (justify mirror))
     )
-    (fp_text value R_Small (at 0 -1.65 90) (layer B.Fab)
+    (fp_text value 10k (at 0 -1.65 90) (layer B.Fab)
       (effects (font (size 1 1) (thickness 0.15)) (justify mirror))
     )
@@
       (effects (font (size 1 1) (thickness 0.15)) (justify mirror))
     )
-    (fp_text value R_Small (at 0 -1.65 90) (layer B.Fab)
+    (fp_text value 220 (at 0 -1.65 90) (layer B.Fab)
       (effects (font (size 1 1) (thickness 0.15)) (justify mirror))
     )
@@
       (effects (font (size 1 1) (thickness 0.15)) (justify mirror))
     )
-    (fp_text value R_Small (at 0 -1.65 90) (layer B.Fab)
+    (fp_text value 220 (at 0 -1.65 90) (layer B.Fab)
       (effects (font (size 1 1) (thickness 0.15)) (justify mirror))
     )
@@
       (effects (font (size 1 1) (thickness 0.15)) (justify mirror))
     )
-    (fp_text value R_Small (at 0 -1.65 90) (layer B.Fab)
+    (fp_text value 220 (at 0 -1.65 90) (layer B.Fab)
       (effects (font (size 1 1) (thickness 0.15)) (justify mirror))
     )
@@
       (effects (font (size 1 1) (thickness 0.15)) (justify mirror))
     )
-    (fp_text value R_Small (at 0 -1.65 90) (layer B.Fab)
+    (fp_text value 220 (at 0 -1.65 90) (layer B.Fab)
       (effects (font (size 1 1) (thickness 0.15)) (justify mirror))
     )
@@
       (effects (font (size 1 1) (thickness 0.15)) (justify mirror))
     )
-    (fp_text value LED_Small (at 0 -1.65) (layer B.Fab)
+    (fp_text value Green (at 0 -1.65) (layer B.Fab)
       (effects (font (size 1 1) (thickness 0.15)) (justify mirror))
     )
@@
       (effects (font (size 1 1) (thickness 0.15)) (justify mirror))
     )
-    (fp_text value LED_Small (at 0 -1.65) (layer B.Fab)
+    (fp_text value Green (at 0 -1.65) (layer B.Fab)
       (effects (font (size 1 1) (thickness 0.15)) (justify mirror))
     )
@@
       (effects (font (size 1 1) (thickness 0.15)) (justify mirror))
     )
-    (fp_text value LED_Small (at 0 -1.65) (layer B.Fab)
+    (fp_text value Green (at 0 -1.65) (layer B.Fab)
       (effects (font (size 1 1) (thickness 0.15)) (justify mirror))
     )
@@
       (effects (font (size 1 1) (thickness 0.15)) (justify mirror))
     )
-    (fp_text value LED_Small (at 0 -1.65) (layer B.Fab)
-      (effects (font (size 1 1) (thickness 0.15)) (justify mirror))
-    )
+    (fp_text value Green (at 0 -1.65) (layer B.Fab)
+      (effects (font (size 1 1) (thickness 0.15)) (justify mirror))
+    )

Commit message: Updated
Parts:
- moved J3 8.16 mm to (256.0, 142.8), turned to 180 degrees
- moved J2 7.82 mm to (236.7, 142.8), turned to 180 degrees
- moved J1 7.47 mm to (217.5, 142.8), turned to 180 degrees
Connections:
- C3 pad 1: Net-(C3-Pad1) -> /FTDI_Controller/USB_DM
- C4 pad 1: Net-(C4-Pad1) -> /FTDI_Controller/USB_DP
- J4 pad 2: Net-(C4-Pad1) -> /FTDI_Controller/USB_DM
- J4 pad 3: Net-(C3-Pad1) -> /FTDI_Controller/USB_DP
- Q1 pad 1: GND -> Net-(Q1-Pad1)
- Q1 pad 2: Net-(Q1-Pad2) -> GND
- Q2 pad 1: GND -> Net-(Q2-Pad1)
- Q2 pad 2: Net-(Q2-Pad2) -> GND
- Q3 pad 1: GND -> Net-(Q3-Pad1)
- Q3 pad 2: Net-(Q3-Pad2) -> GND
- Q4 pad 1: GND -> Net-(Q4-Pad1)
- Q4 pad 2: Net-(Q4-Pad2) -> GND
- R10 pad 2: Net-(C4-Pad1) -> /FTDI_Controller/USB_DP
- R5 pad 1: Net-(Q1-Pad2) -> Net-(Q1-Pad1)
- R6 pad 1: Net-(Q2-Pad2) -> Net-(Q2-Pad1)
- R7 pad 1: Net-(Q3-Pad2) -> Net-(Q3-Pad1)
- R8 pad 1: Net-(Q4-Pad2) -> Net-(Q4-Pad1)
- R9 pad 2: Net-(C3-Pad1) -> /FTDI_Controller/USB_DM
Routing:
- net GND: track 15.2 -> 46.6 mm
- net Net-(C4-Pad1): track 17.7 -> 0.00 mm, vias 1 -> 0
- net /FTDI_Controller/USB_DM: track 0.00 -> 13.7 mm, vias 0 -> 1
- net /FTDI_Controller/USB_DP: track 0.00 -> 13.2 mm, vias 0 -> 1
- net Net-(C3-Pad1): track 9.68 -> 0.00 mm, vias 1 -> 0
- net Net-(Q4-Pad2): track 5.67 -> 0.00 mm
- net Net-(Q2-Pad2): track 5.15 -> 0.00 mm
- net Net-(Q1-Pad2): track 5.13 -> 0.00 mm
- net Net-(Q3-Pad2): track 5.12 -> 0.00 mm
- net Net-(Q2-Pad1): track 0.00 -> 2.63 mm
- net Net-(Q1-Pad1): track 0.00 -> 2.61 mm
- net Net-(Q3-Pad1): track 0.00 -> 2.60 mm
- net Net-(Q4-Pad1): track 0.00 -> 2.55 mm
