File: hw/v0p1/NetworkBreaker.sch (KiCad schematic (older format))
At the start: 32 parts, among them J1 8P8C_Shielded, J2 8P8C_Shielded, J3 8P8C_Shielded, K1 M4-5HAW, K2 M4-5HAW, K3 M4-5HAW, K4 M4-5HAW, Q1 2N3904, Q2 2N3904, Q3 2N3904, Q4 2N3904, U1 TLP627-4

Commit message: Updated BOM
Parts:
- D1, D2, D3, D4: value LED_Small -> Green; LCSC (none) -> C125090
- R1, R2, R3, R4: value R_Small -> 220; LCSC (none) -> C413172
- R5, R6, R7, R8: value R_Small -> 10k; LCSC (none) -> C180849
Changed lines of the file:
@@
 P 5000 1650
 F 0 "R2" V 4804 1650 50  0000 C CNN
-F 1 "R_Small" V 4895 1650 50  0000 C CNN
+F 1 "220" V 4895 1650 50  0000 C CNN
 F 2 "Resistor_SMD:R_0805_2012Metric" H 5000 1650 50  0001 C CNN
 F 3 "~" H 5000 1650 50  0001 C CNN
+F 4 "C413172" V 5000 1650 50  0001 C CNN "LCSC"
 	1    5000 1650
 	0    1    1    0
@@
 P 5000 3250
 F 0 "R3" V 4804 3250 50  0000 C CNN
-F 1 "R_Small" V 4895 3250 50  0000 C CNN
+F 1 "220" V 4895 3250 50  0000 C CNN
 F 2 "Resistor_SMD:R_0805_2012Metric" H 5000 3250 50  0001 C CNN
 F 3 "~" H 5000 3250 50  0001 C CNN
+F 4 "C413172" V 5000 3250 50  0001 C CNN "LCSC"
 	1    5000 3250
 	0    1    1    0
@@
 P 5000 4850
 F 0 "R4" V 4804 4850 50  0000 C CNN
-F 1 "R_Small" V 4895 4850 50  0000 C CNN
+F 1 "220" V 4895 4850 50  0000 C CNN
 F 2 "Resistor_SMD:R_0805_2012Metric" H 5000 4850 50  0001 C CNN
 F 3 "~" H 5000 4850 50  0001 C CNN
+F 4 "C413172" V 5000 4850 50  0001 C CNN "LCSC"
 	1    5000 4850
 	0    1    1    0
@@
 P 4950 6450
 F 0 "R1" V 4754 6450 50  0000 C CNN
-F 1 "R_Small" V 4845 6450 50  0000 C CNN
+F 1 "220" V 4845 6450 50  0000 C CNN
 F 2 "Resistor_SMD:R_0805_2012Metric" H 4950 6450 50  0001 C CNN
 F 3 "~" H 4950 6450 50  0001 C CNN
+F 4 "C413172" V 4950 6450 50  0001 C CNN "LCSC"
 	1    4950 6450
 	0    1    1    0
@@
 P 5000 1850
 F 0 "D2" H 5000 2085 50  0000 C CNN
-F 1 "LED_Small" H 5000 1994 50  0000 C CNN
+F 1 "Green" H 5000 1994 50  0000 C CNN
 F 2 "LED_SMD:LED_0805_2012Metric" V 5000 1850 50  0001 C CNN
 F 3 "~" V 5000 1850 50  0001 C CNN
+F 4 " C125090" H 5000 1850 50  0001 C CNN "LCSC"
 	1    5000 1850
 	1    0    0    -1
@@
 P 5000 3450
 F 0 "D3" H 5000 3685 50  0000 C CNN
-F 1 "LED_Small" H 5000 3594 50  0000 C CNN
+F 1 "Green" H 5000 3594 50  0000 C CNN
 F 2 "LED_SMD:LED_0805_2012Metric" V 5000 3450 50  0001 C CNN
 F 3 "~" V 5000 3450 50  0001 C CNN
+F 4 " C125090" H 5000 3450 50  0001 C CNN "LCSC"
 	1    5000 3450
 	1    0    0    -1
@@
 P 5000 5050
 F 0 "D4" H 5000 5285 50  0000 C CNN
-F 1 "LED_Small" H 5000 5194 50  0000 C CNN
+F 1 "Green" H 5000 5194 50  0000 C CNN
 F 2 "LED_SMD:LED_0805_2012Metric" V 5000 5050 50  0001 C CNN
 F 3 "~" V 5000 5050 50  0001 C CNN
+F 4 " C125090" H 5000 5050 50  0001 C CNN "LCSC"
 	1    5000 5050
 	1    0    0    -1
@@
 P 4950 6650
 F 0 "D1" H 4950 6885 50  0000 C CNN
-F 1 "LED_Small" H 4950 6794 50  0000 C CNN
+F 1 "Green" H 4950 6794 50  0000 C CNN
 F 2 "LED_SMD:LED_0805_2012Metric" V 4950 6650 50  0001 C CNN
 F 3 "~" V 4950 6650 50  0001 C CNN
+F 4 " C125090" H 4950 6650 50  0001 C CNN "LCSC"
 	1    4950 6650
 	1    0    0    -1
@@
 P 6250 3450
 F 0 "R7" V 6054 3450 50  0000 C CNN
-F 1 "R_Small" V 6145 3450 50  0000 C CNN
+F 1 "10k" V 6145 3450 50  0000 C CNN
 F 2 "Resistor_SMD:R_0805_2012Metric" H 6250 3450 50  0001 C CNN
 F 3 "~" H 6250 3450 50  0001 C CNN
+F 4 "C180849" V 6250 3450 50  0001 C CNN "LCSC"
 	1    6250 3450
 	0    1    1    0
@@
 P 6250 5050
 F 0 "R8" V 6054 5050 50  0000 C CNN
-F 1 "R_Small" V 6145 5050 50  0000 C CNN
+F 1 "10k" V 6145 5050 50  0000 C CNN
 F 2 "Resistor_SMD:R_0805_2012Metric" H 6250 5050 50  0001 C CNN
 F 3 "~" H 6250 5050 50  0001 C CNN
+F 4 "C180849" V 6250 5050 50  0001 C CNN "LCSC"
 	1    6250 5050
 	0    1    1    0
@@
 P 6250 1850
 F 0 "R6" V 6054 1850 50  0000 C CNN
-F 1 "R_Small" V 6145 1850 50  0000 C CNN
+F 1 "10k" V 6145 1850 50  0000 C CNN
 F 2 "Resistor_SMD:R_0805_2012Metric" H 6250 1850 50  0001 C CNN
 F 3 "~" H 6250 1850 50  0001 C CNN
+F 4 "C180849" V 6250 1850 50  0001 C CNN "LCSC"
 	1    6250 1850
 	0    1    1    0
@@
 P 6200 6650
 F 0 "R5" V 6004 6650 50  0000 C CNN
-F 1 "R_Small" V 6095 6650 50  0000 C CNN
+F 1 "10k" V 6095 6650 50  0000 C CNN
 F 2 "Resistor_SMD:R_0805_2012Metric" H 6200 6650 50  0001 C CNN
 F 3 "~" H 6200 6650 50  0001 C CNN
+F 4 "C180849" V 6200 6650 50  0001 C CNN "LCSC"
 	1    6200 6650
 	0    1    1    0

Commit message: Updated part LCSC part numbers
Parts:
- U1: symbol Isolator:TLP627-4 -> Isolator:LTV-847M
- U1: symbol Isolator:TLP627-4 -> Isolator:LTV-847M; LCSC C89243 -> C13497
Connections:
- wire segments 106 -> 110
Changed lines of the file:
@@
 Mounting Holes
 $Comp
-L Isolator:TLP627-4 U1
+L Isolator:LTV-847M U1
 U 2 1 5F40E333
 P 5650 4950
@@
 $EndComp
 $Comp
-L Isolator:TLP627-4 U1
+L Isolator:LTV-847M U1
 U 4 1 5F41365E
 P 5650 1750
@@
 $EndComp
 $Comp
-L Isolator:TLP627-4 U1
+L Isolator:LTV-847M U1
 U 1 1 5F415A77
 P 5600 6550
@@
 	0    1    1    0
 $EndComp
-Wire Wire Line
-	5100 1650 5250 1650
-Wire Wire Line
-	5100 3250 5250 3250
-Wire Wire Line
-	5100 4850 5250 4850
-Wire Wire Line
-	5050 6450 5200 6450
 $Comp
 L power:GND #PWR04
@@
 $EndComp
 Wire Wire Line
-	5250 1850 5100 1850
-Wire Wire Line
 	4900 1850 4650 1850
 Wire Wire Line
 	4650 1850 4650 1900
 Wire Wire Line
-	5250 3450 5100 3450
-Wire Wire Line
 	4900 3450 4700 3450
 Wire Wire Line
@@
 Wire Wire Line
 	4700 5050 4700 5100
-Wire Wire Line
-	5100 5050 5250 5050
-Wire Wire Line
-	5200 6650 5050 6650
 Wire Wire Line
 	4850 6650 4650 6650
@@
 Wire Wire Line
 	6000 6400 6000 6450
-Wire Wire Line
-	6050 3450 6150 3450
 $Comp
 L Transistor_BJT:2N3904 Q3
@@
 Wire Wire Line
 	6050 4800 6050 4850
-Wire Wire Line
-	6050 5050 6150 5050
 $Comp
 L Transistor_BJT:2N3904 Q4
@@
 Wire Wire Line
 	6050 1600 6050 1650
-Wire Wire Line
-	6050 1850 6150 1850
 $Comp
 L Transistor_BJT:2N3904 Q2
@@
 	1    0    0    -1
 $EndComp
-Wire Wire Line
-	6000 6650 6100 6650
 $Comp
 L Transistor_BJT:2N3904 Q1
@@
 	4600 6450 4850 6450
 $Comp
-L Isolator:TLP627-4 U1
+L Isolator:LTV-847M U1
 U 3 1 5F412367
 P 5650 3350
@@
 F 2 "Package_DIP:DIP-16_W7.62mm" H 5350 3150 50  0001 L CIN
 F 3 "https://toshiba.semicon-storage.com/info/docget.jsp?did=16914&prodName=TLP627" H 5650 3350 50  0001 L CNN
-F 4 "C89243" H 5650 3350 50  0001 C CNN "LCSC"
+F 4 "C13497" H 5650 3350 50  0001 C CNN "LCSC"
 	3    5650 3350
 	1    0    0    -1
 $EndComp
+Wire Wire Line
+	6050 1650 5950 1650
+Wire Wire Line
+	5950 1850 6150 1850
+Wire Wire Line
+	5100 1850 5350 1850
+Wire Wire Line
+	5100 1650 5350 1650
+Wire Wire Line
+	5100 3250 5350 3250
+Wire Wire Line
+	5100 3450 5350 3450
+Wire Wire Line
+	6050 3250 5950 3250
+Wire Wire Line
+	5950 3450 6150 3450
+Wire Wire Line
+	5100 4850 5350 4850
+Wire Wire Line
+	5100 5050 5350 5050
+Wire Wire Line
+	5950 4850 6050 4850
+Wire Wire Line
+	5950 5050 6150 5050
+Wire Wire Line
+	5900 6450 6000 6450
+Wire Wire Line
+	5050 6650 5300 6650
+Wire Wire Line
+	5050 6450 5300 6450
+Wire Wire Line
+	5900 6650 6100 6650
 $EndSCHEMATC

Commit message: Updated
Parts:
- Q1, Q2, Q3, Q4: symbol Transistor_BJT:2N3904 -> Transistor_BJT:BC818
Other:
- note added: "B"
- note added: "B 1"
- note added: "C"
- note added: "C 3"
- note added: "E"
- note added: "E 2"
Changed lines of the file:
@@
 	6000 6400 6000 6450
 $Comp
-L Transistor_BJT:2N3904 Q3
+L Transistor_BJT:BC818 Q3
 U 1 1 5F46B1C0
 P 6550 3450
@@
 	6050 4800 6050 4850
 $Comp
-L Transistor_BJT:2N3904 Q4
+L Transistor_BJT:BC818 Q4
 U 1 1 5F4B54C4
 P 6550 5050
@@
 	6050 1600 6050 1650
 $Comp
-L Transistor_BJT:2N3904 Q2
+L Transistor_BJT:BC818 Q2
 U 1 1 5F4BA1BF
 P 6550 1850
@@
 $EndComp
 $Comp
-L Transistor_BJT:2N3904 Q1
+L Transistor_BJT:BC818 Q1
 U 1 1 5F4E2F7F
 P 6500 6650
@@
 Wire Wire Line
 	5900 6650 6100 6650
+Text Notes 6400 1850 0    50   ~ 0
+B
+Text Notes 6550 1700 0    50   ~ 0
+C
+Text Notes 6550 2050 0    50   ~ 0
+E
+Wire Notes Line
+	6200 850  6200 1050
+Wire Notes Line
+	6200 1050 5800 1050
+Wire Notes Line
+	5800 1050 5800 850
+Wire Notes Line
+	5950 850  5950 750
+Wire Notes Line
+	5950 750  6050 750
+Wire Notes Line
+	6050 750  6050 850
+Wire Notes Line
+	5800 850  6200 850
+Wire Notes Line
+	6150 1050 6150 1150
+Wire Notes Line
+	6150 1150 6050 1150
+Wire Notes Line
+	6050 1150 6050 1050
+Wire Notes Line
+	5850 1050 5850 1150
+Wire Notes Line
+	5850 1150 5950 1150
+Wire Notes Line
+	5950 1150 5950 1050
+Text Notes 5950 750  0    50   ~ 0
+C 3
+Text Notes 6100 1250 0    50   ~ 0
+E 2
+Text Notes 5850 1250 0    50   ~ 0
+B 1
 $EndSCHEMATC
