File: hw/v0p2/FTDI_Controller.sch (KiCad schematic (older format))
At the start: 12 parts, among them J4 USB_B_Micro, J5 Conn_01x06, U2 FT230XS

Commit message: Updated
Parts:
- renumbered C6 to C5, C5 to C6, R9 to R4, R10 to R5
Connections:
- net labels added: CBUS0, CBUS1, CBUS2, CBUS3
- net labels removed: GPIO13, GPIO19, GPIO5, GPIO6
- wire segments 45 -> 47
- no-connect marks 1 -> 2
Other:
- note removed: "These signal names don't make any sense \nhere. These are the RPi names for when the \nraspberry pi is used."
Changed lines of the file:
@@
 $Descr A4 11693 8268
 encoding utf-8
-Sheet 3 3
+Sheet 3 5
 Title ""
 Date ""
@@
 $EndComp
 $Comp
-L power:GND #PWR026
+L power:GND #PWR013
 U 1 1 5F61889B
 P 4200 2650
-F 0 "#PWR026" H 4200 2400 50  0001 C CNN
+F 0 "#PWR013" H 4200 2400 50  0001 C CNN
 F 1 "GND" H 4205 2477 50  0000 C CNN
 F 2 "" H 4200 2650 50  0001 C CNN
@@
 $EndComp
 $Comp
-L power:GND #PWR027
+L power:GND #PWR014
 U 1 1 5F618E39
 P 4300 2650
-F 0 "#PWR027" H 4300 2400 50  0001 C CNN
+F 0 "#PWR014" H 4300 2400 50  0001 C CNN
 F 1 "GND" H 4305 2477 50  0000 C CNN
 F 2 "" H 4300 2650 50  0001 C CNN
@@
 $EndComp
 $Comp
-L power:GND #PWR033
+L power:GND #PWR019
 U 1 1 5F618F68
 P 6350 3900
-F 0 "#PWR033" H 6350 3650 50  0001 C CNN
+F 0 "#PWR019" H 6350 3650 50  0001 C CNN
 F 1 "GND" H 6355 3727 50  0000 C CNN
 F 2 "" H 6350 3900 50  0001 C CNN
@@
 $EndComp
 $Comp
-L power:GND #PWR034
+L power:GND #PWR0101
 U 1 1 5F61925E
 P 6550 3900
-F 0 "#PWR034" H 6550 3650 50  0001 C CNN
+F 0 "#PWR0101" H 6550 3650 50  0001 C CNN
 F 1 "GND" H 6555 3727 50  0000 C CNN
 F 2 "" H 6550 3900 50  0001 C CNN
@@
 $EndComp
 $Comp
-L Device:R_Small R9
+L Device:R_Small R4
 U 1 1 5F62D59A
 P 5550 2850
-F 0 "R9" V 5354 2850 50  0000 C CNN
+F 0 "R4" V 5354 2850 50  0000 C CNN
 F 1 "27" V 5445 2850 50  0000 C CNN
 F 2 "Resistor_SMD:R_0805_2012Metric" H 5550 2850 50  0001 C CNN
@@
 $EndComp
 $Comp
-L Device:R_Small R10
+L Device:R_Small R5
 U 1 1 5F62E0D2
 P 5550 2950
-F 0 "R10" V 5750 2950 50  0000 C CNN
+F 0 "R5" V 5750 2950 50  0000 C CNN
 F 1 "27" V 5650 2950 50  0000 C CNN
 F 2 "Resistor_SMD:R_0805_2012Metric" H 5550 2950 50  0001 C CNN
@@
 $EndComp
 $Comp
-L Device:C_Small C6
+L Device:C_Small C5
 U 1 1 5F62F1D7
 P 5500 2100
-F 0 "C6" H 5592 2146 50  0000 L CNN
+F 0 "C5" H 5592 2146 50  0000 L CNN
 F 1 "10nF" H 5592 2055 50  0000 L CNN
 F 2 "Capacitor_SMD:C_0805_2012Metric" H 5500 2100 50  0001 C CNN
@@
 	6550 2250 7100 2250
 $Comp
-L power:+5V #PWR032
+L power:+5V #PWR018
 U 1 1 5F6353FA
 P 6350 2000
-F 0 "#PWR032" H 6350 1850 50  0001 C CNN
+F 0 "#PWR018" H 6350 1850 50  0001 C CNN
 F 1 "+5V" H 6365 2173 50  0000 C CNN
 F 2 "" H 6350 2000 50  0001 C CNN
@@
 $EndComp
 $Comp
-L power:+5V #PWR024
+L power:+5V #PWR011
 U 1 1 5F63662A
 P 4000 3550
-F 0 "#PWR024" H 4000 3400 50  0001 C CNN
+F 0 "#PWR011" H 4000 3400 50  0001 C CNN
 F 1 "+5V" H 4015 3723 50  0000 C CNN
 F 2 "" H 4000 3550 50  0001 C CNN
@@
 $EndComp
 $Comp
-L power:GND #PWR025
+L power:GND #PWR012
 U 1 1 5F636E8E
 P 4000 3900
-F 0 "#PWR025" H 4000 3650 50  0001 C CNN
+F 0 "#PWR012" H 4000 3650 50  0001 C CNN
 F 1 "GND" H 4005 3727 50  0000 C CNN
 F 2 "" H 4000 3900 50  0001 C CNN
@@
 $EndComp
 $Comp
-L power:GND #PWR028
+L power:GND #PWR015
 U 1 1 5F63EB83
 P 5000 2650
-F 0 "#PWR028" H 5000 2400 50  0001 C CNN
+F 0 "#PWR015" H 5000 2400 50  0001 C CNN
 F 1 "GND" H 5005 2477 50  0000 C CNN
 F 2 "" H 5000 2650 50  0001 C CNN
@@
 $EndComp
 $Comp
-L power:GND #PWR029
+L power:GND #PWR016
 U 1 1 5F63F10D
 P 5000 3150
-F 0 "#PWR029" H 5000 2900 50  0001 C CNN
+F 0 "#PWR016" H 5000 2900 50  0001 C CNN
 F 1 "GND" H 5005 2977 50  0000 C CNN
 F 2 "" H 5000 3150 50  0001 C CNN
@@
 Connection ~ 5000 2950
 $Comp
-L Device:C_Small C5
+L Device:C_Small C6
 U 1 1 5F640973
 P 7600 4350
-F 0 "C5" H 7692 4396 50  0000 L CNN
+F 0 "C6" H 7692 4396 50  0000 L CNN
 F 1 "100nF" H 7692 4305 50  0000 L CNN
 F 2 "Capacitor_SMD:C_0805_2012Metric" H 7600 4350 50  0001 C CNN
@@
 	7050 4150 7600 4150
 $Comp
-L power:GND #PWR030
+L power:GND #PWR0102
 U 1 1 5F64542D
 P 7600 4550
-F 0 "#PWR030" H 7600 4300 50  0001 C CNN
+F 0 "#PWR0102" H 7600 4300 50  0001 C CNN
 F 1 "GND" H 7605 4377 50  0000 C CNN
 F 2 "" H 7600 4550 50  0001 C CNN
@@
 Wire Wire Line
 	3800 3900 4000 3900
-Text Notes 7200 3600 0    50   ~ 0
-These signal names don't make any sense \nhere. These are the RPi names for when the \nraspberry pi is used.
 $Comp
 L Connector_Generic:Conn_01x06 J5
@@
 	7150 2850 8050 2850
 $Comp
-L power:+5V #PWR035
+L power:+5V #PWR0103
 U 1 1 5F650F75
 P 7850 2350
-F 0 "#PWR035" H 7850 2200 50  0001 C CNN
+F 0 "#PWR0103" H 7850 2200 50  0001 C CNN
 F 1 "+5V" V 7865 2478 50  0000 L CNN
 F 2 "" H 7850 2350 50  0001 C CNN
@@
 $EndComp
 $Comp
-L power:GND #PWR036
+L power:GND #PWR0104
 U 1 1 5F651A4F
 P 7850 2450
-F 0 "#PWR036" H 7850 2200 50  0001 C CNN
+F 0 "#PWR0104" H 7850 2200 50  0001 C CNN
 F 1 "GND" V 7855 2322 50  0000 R CNN
 F 2 "" H 7850 2450 50  0001 C CNN
@@
 	5500 2000 5800 2000
 $Comp
-L power:GND #PWR031
+L power:GND #PWR017
 U 1 1 5F6574CA
 P 5500 2200
-F 0 "#PWR031" H 5500 1950 50  0001 C CNN
+F 0 "#PWR017" H 5500 1950 50  0001 C CNN
 F 1 "GND" H 5505 2027 50  0000 C CNN
 F 2 "" H 5500 2200 50  0001 C CNN
@@
 Circuit copied from FTDI data sheet, section 7.1\nhttps://datasheet.lcsc.com/szlcsc/1811151642_FTDI-Future-Designs-FT230XS-R_C69082.pdf
 Text GLabel 7350 3250 2    50   Input ~ 0
-GPIO13
+CBUS2
 Text GLabel 7350 3350 2    50   Input ~ 0
-GPIO19
+CBUS3
 Text GLabel 7350 3150 2    50   Input ~ 0
-GPIO6
+CBUS1
 Text GLabel 7350 3050 2    50   Input ~ 0
-GPIO5
+CBUS0
 Wire Wire Line
 	7150 3350 7350 3350
@@
 Wire Wire Line
 	4600 2200 4950 2200
+NoConn ~ 8250 2600
+Wire Wire Line
+	8700 3300 9600 3300
+Wire Wire Line
+	8700 3400 9600 3400
+Text Label 8750 3300 0    50   ~ 0
+FTDI_TXD
+Text Label 8750 3400 0    50   ~ 0
+FTDI_RXD
+Text GLabel 9600 3400 2    50   Input ~ 0
+FTDI_RXD
+Text GLabel 9600 3300 2    50   Input ~ 0
+FTDI_TXD
 $EndSCHEMATC
