File: hw/v0p2/NetworkBreaker.kicad_pcb (KiCad board)
At the start: 2 copper layers, 65 x 56 mm, 45 parts, among them J1 8P8C_Shielded, J2 8P8C_Shielded, J3 8P8C_Shielded, J4 USB_B_Micro, J5 Conn_01x06, K1 M4-5HAW, K2 M4-5HAW, K3 M4-5HAW, K4 M4-5HAW, P1 Conn_02x20_Odd_Even, Q1 2N3904, Q2 2N3904, Q3 2N3904, Q4 2N3904, U1 TLP627-4, U2 FT230XS

Commit message: Updated
Parts:
- removed the C6 at (208.2, 102.9)
- removed D5, D6, D7, D8: D_Small, Diode_SMD:D_SOD-123F
- removed MK4: M2.5, MountingHole:MountingHole_2.7mm_M2.5
- removed Q1, Q2, Q3, Q4: 2N3904, Package_TO_SOT_SMD:SOT-23
- removed the R4 at (244.3, 105.8)
- removed the R5 at (258.6, 115.3)
- added A1: Arduino_Nano_v3.x, Module:Arduino_Nano, F.Cu at (224.9, 122.3)
- added C5: 10nF, Capacitor_SMD:C_0805_2012Metric, B.Cu at (207.8, 102.8)
- added J6: Conn_01x15_Female, Connector_PinSocket_2.54mm:PinSocket_1x15_P2.54mm_Vertical, B.Cu at (224.9, 110.6)
- added J7: Conn_01x15_Female, Connector_PinSocket_2.54mm:PinSocket_1x15_P2.54mm_Vertical, B.Cu at (224.8, 119.3)
- D1, D2, D3, D4: value Green -> LED_Small; moved to F.Cu
- J5: moved to B.Cu
- R1, R2, R3: value 220 -> R_Small
- R6: value 10k -> R_Small
- R7, R8: value 10k -> 0
- U1: value TLP627-4 -> ULN2003; footprint Package_DIP:DIP-16_W7.62mm -> Package_SO:TSSOP-16_4.4x5mm_P0.65mm; moved to B.Cu
- moved J5 52.7 mm to (248.8, 102.5), turned to 270 degrees
- moved K4 45.6 mm to (201.5, 133.0), turned to 0 degrees
- moved U1 43.1 mm to (223.3, 137.2), turned to 0 degrees
- moved R6 41.8 mm to (261.0, 138.1), turned to 270 degrees
- moved D4 39.4 mm to (263.4, 143.1), turned to 90 degrees
- moved D3 34.1 mm to (263.4, 139.7), turned to 90 degrees
- moved R2 33.2 mm to (245.4, 137.0), turned to 0 degrees
- moved R3 32.9 mm to (249.6, 137.0), turned to 0 degrees
- moved R1 32.3 mm to (241.1, 137.0), turned to 0 degrees
- moved K3 31.6 mm to (201.5, 122.4), turned to 0 degrees
- moved D1 31.2 mm to (263.4, 132.9), turned to 90 degrees
- moved D2 28.7 mm to (263.4, 136.3), turned to 90 degrees
- moved K1 22.1 mm to (243.1, 133.0), turned to 0 degrees
- moved R7 22.1 mm to (258.8, 113.3), turned to 180 degrees
- moved K2 19.4 mm to (222.3, 133.0), turned to 0 degrees
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- renumbered C5 to C6, R9 to R4, R10 to R5
Connections:
- net /ENET1_PIN1 renamed ENET1_PIN1
- net /ENET1_PIN2 renamed ENET1_PIN2
- net /ENET1_PIN5 renamed ENET1_PIN5
- net /ENET1_PIN6 renamed ENET1_PIN6
- net /ENET2_PIN1 renamed ENET2_PIN1
- net /ENET2_PIN2 renamed ENET2_PIN2
- net /ENET2_PIN5 renamed ENET2_PIN5
- net /ENET2_PIN6 renamed ENET2_PIN6
- net /ENET3_PIN1 renamed ENET3_PIN1
- net /ENET3_PIN2 renamed ENET3_PIN2
- net /ENET3_PIN5 renamed ENET3_PIN5
- net /ENET3_PIN6 renamed ENET3_PIN6
- net /FTDI_Controller/FTDI_RXD renamed FTDI_RXD
- net /FTDI_Controller/FTDI_TXD renamed FTDI_TXD
- D1 pad 1: GND -> Net-(D1-Pad1)
- D1 pad 2: Net-(D1-Pad2) -> +5V
- D2 pad 1: GND -> Net-(D2-Pad1)
- D2 pad 2: Net-(D2-Pad2) -> +5V
- D3 pad 1: GND -> Net-(D3-Pad1)
- D3 pad 2: Net-(D3-Pad2) -> +5V
- D4 pad 1: GND -> Net-(D4-Pad1)
- D4 pad 2: Net-(D4-Pad2) -> +5V
- J1 pad 3: /ENET1_PIN3 -> ENET1_PIN3
- J1 pad 4: /ENET1_PIN4 -> ENET1_PIN4
- J1 pad 7: /ENET1_PIN7 -> ENET1_PIN7
- J1 pad 8: /ENET1_PIN8 -> ENET1_PIN8
- J2 pad 3: /ENET2_PIN3 -> ENET2_PIN3
- J2 pad 4: /ENET2_PIN4 -> ENET2_PIN4
- J2 pad 7: /ENET2_PIN7 -> ENET2_PIN7
- J2 pad 8: /ENET2_PIN8 -> ENET2_PIN8
- J3 pad 3: /ENET3_PIN3 -> ENET3_PIN3
- J3 pad 4: /ENET3_PIN4 -> ENET3_PIN4
- J3 pad 7: /ENET3_PIN7 -> ENET3_PIN7
- J3 pad 8: /ENET3_PIN8 -> ENET3_PIN8
- J4 pad 4: (no net) -> Net-(J4-Pad4)
- K1 pad A2: Net-(D5-Pad2) -> RELAY_4_CTRL
- K2 pad 11: /ENET1_PIN8 -> ENET1_PIN4
- K2 pad 12: /ENET2_PIN8 -> ENET2_PIN4
- K2 pad 14: /ENET3_PIN8 -> ENET3_PIN4
- K2 pad 21: /ENET1_PIN7 -> ENET1_PIN3
- K2 pad 22: /ENET2_PIN7 -> ENET2_PIN3
- K2 pad 24: /ENET3_PIN7 -> ENET3_PIN3
- K2 pad A2: Net-(D6-Pad2) -> RELAY_3_CTRL
- K3 pad A2: Net-(D7-Pad2) -> RELAY_2_CTRL
- K4 pad 11: /ENET1_PIN4 -> ENET1_PIN8
- K4 pad 12: /ENET2_PIN4 -> ENET2_PIN8
- K4 pad 14: /ENET3_PIN4 -> ENET3_PIN8
- K4 pad 21: /ENET1_PIN3 -> ENET1_PIN7
- K4 pad 22: /ENET2_PIN3 -> ENET2_PIN7
- K4 pad 24: /ENET3_PIN3 -> ENET3_PIN7
- K4 pad A2: Net-(D8-Pad2) -> RELAY_1_CTRL
- P1 pad 10: (no net) -> /RPi_Connector/GPIO15(RXD0)
- P1 pad 11: (no net) -> /RPi_Connector/GPIO17(GEN0)
- P1 pad 12: (no net) -> /RPi_Connector/GPIO18(GEN1)(PWM0)
- P1 pad 13: (no net) -> /RPi_Connector/GPIO27(GEN2)
- P1 pad 15: (no net) -> /RPi_Connector/GPIO22(GEN3)
- P1 pad 16: (no net) -> /RPi_Connector/GPIO23(GEN4)
- P1 pad 18: (no net) -> /RPi_Connector/GPIO24(GEN5)
- P1 pad 19: (no net) -> /RPi_Connector/GPIO10(SPI0_MOSI)
- P1 pad 21: (no net) -> /RPi_Connector/GPIO9(SPI0_MISO)
- P1 pad 22: (no net) -> /RPi_Connector/GPIO25(GEN6)
- P1 pad 23: (no net) -> /RPi_Connector/GPIO11(SPI0_SCK)
- P1 pad 24: (no net) -> /RPi_Connector/GPIO8(SPI0_CE_N)
- P1 pad 26: (no net) -> /RPi_Connector/GPIO7(SPI1_CE_N)
- P1 pad 27: (no net) -> /RPi_Connector/ID_SD
- P1 pad 28: (no net) -> /RPi_Connector/ID_SC
- P1 pad 29: GPIO5 -> CBUS0
- P1 pad 3: (no net) -> /RPi_Connector/GPIO2(SDA1)
- P1 pad 31: GPIO6 -> CBUS1
- P1 pad 32: (no net) -> /RPi_Connector/GPIO12(PWM0)
- P1 pad 33: GPIO13 -> CBUS2
- P1 pad 35: GPIO19 -> CBUS3
- P1 pad 36: (no net) -> /RPi_Connector/GPIO16
- P1 pad 37: (no net) -> /RPi_Connector/GPIO26
- P1 pad 38: (no net) -> /RPi_Connector/GPIO20(SPI1_MOSI)
- P1 pad 40: (no net) -> /RPi_Connector/GPIO21(SPI1_SCK)
- P1 pad 5: (no net) -> /RPi_Connector/GPIO3(SCL1)
- P1 pad 7: (no net) -> /RPi_Connector/GPIO4(GCLK)
- P1 pad 8: (no net) -> /RPi_Connector/GPIO14(TXD0)
- R1 pad 1: Net-(R1-Pad1) -> LED_1_CTRL
- R1 pad 2: GPIO19 -> Net-(D1-Pad1)
- R2 pad 1: Net-(R2-Pad1) -> LED_2_CTRL
- R2 pad 2: GPIO5 -> Net-(D2-Pad1)
- R3 pad 1: Net-(R3-Pad1) -> LED_3_CTRL
- R3 pad 2: GPIO6 -> Net-(D3-Pad1)
- R6 pad 1: Net-(Q2-Pad1) -> GND
- R6 pad 2: Net-(R6-Pad2) -> Net-(D4-Pad1)
- R7 pad 1: Net-(Q3-Pad1) -> +3V3
- R7 pad 2: Net-(R7-Pad2) -> ARD_3p3v
- R8 pad 1: Net-(Q4-Pad1) -> ARD_5v
- R8 pad 2: Net-(R8-Pad2) -> +5V
- U1 pad 1: Net-(R1-Pad1) -> CBUS0
- U1 pad 10: +5V -> LED_3_CTRL
- U1 pad 11: Net-(R7-Pad2) -> LED_2_CTRL
- U1 pad 12: +5V -> LED_1_CTRL
- U1 pad 13: Net-(R8-Pad2) -> RELAY_4_CTRL
- U1 pad 14: +5V -> RELAY_3_CTRL
- U1 pad 15: Net-(R5-Pad2) -> RELAY_2_CTRL
- U1 pad 16: +5V -> RELAY_1_CTRL
- U1 pad 2: Net-(D1-Pad2) -> CBUS0
- U1 pad 3: Net-(R4-Pad1) (its old number) -> CBUS0
- U1 pad 4: Net-(D4-Pad2) -> CBUS0
- U1 pad 5: Net-(R3-Pad1) -> CBUS1
- U1 pad 6: Net-(D3-Pad2) -> CBUS2
- U1 pad 7: Net-(R2-Pad1) -> CBUS3
- U1 pad 8: Net-(D2-Pad2) -> GND
- U1 pad 9: Net-(R6-Pad2) -> +5V
- U2 pad 14: GPIO6 -> CBUS1
- U2 pad 15: GPIO5 -> CBUS0
- U2 pad 16: GPIO19 -> CBUS3
- U2 pad 7: GPIO13 -> CBUS2
Routing:
- net CBUS3: track 0.00 -> 93.1 mm, vias 0 -> 3
- net CBUS2: track 0.00 -> 92.4 mm, vias 0 -> 4
- net CBUS1: track 0.00 -> 92.1 mm, vias 0 -> 4
- net CBUS0: track 0.00 -> 85.4 mm, vias 0 -> 4
- net /ENET1_PIN4: track 61.4 -> 0.00 mm, vias 1 -> 0
- net +5V: track 139.4 -> 200.6 mm, vias 1 -> 6
- net /ENET1_PIN3: track 58.5 -> 0.00 mm, vias 1 -> 0
- net GND: track 46.6 -> 99.5 mm, vias 19 -> 15
- net GPIO13: track 51.8 -> 0.00 mm, vias 4 -> 0
- net RELAY_2_CTRL: track 0.00 -> 50.7 mm, vias 0 -> 2
- net /ENET3_PIN8: track 46.9 -> 0.00 mm, vias 1 -> 0
- net +3V3: track 21.4 -> 67.6 mm, vias 0 -> 1
- net GPIO19: track 45.1 -> 0.00 mm, vias 2 -> 0
- net ENET3_PIN7: track 0.00 -> 44.8 mm, vias 0 -> 2
- net FTDI_RXD: track 19.8 -> 63.2 mm, vias 0 -> 2
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Other:
- board text added: "RX"
- board text added: "TX"
- board text removed: "Copyright (C) 2020 A. Kuker Version 0.1"
- board text removed: "RXD"
- board text removed: "TXD"
