File: hw/v1p0/NetworkBreaker.sch (KiCad schematic (older format))
At the start: 15 parts, among them J1 8P8C_Shielded, J2 8P8C_Shielded, K1 M4-5HAW, K2 M4-5HAW, K3 M4-5HAW, K4 M4-5HAW, U1 ULN2003

Commit message: Updated
Parts:
- removed D1, D2, D3, D4: LED_Small, LED_SMD:LED_0805_2012Metric, symbol Device:LED_Small
- removed K1, K2, K3, K4: M4-5HAW, Relay_THT:Relay_DPDT_Finder_30.22, symbol Relay:FINDER-30.22
- removed R1, R2, R3, R6: R_Small, Resistor_SMD:R_0805_2012Metric, symbol Device:R_Small
- removed U1: ULN2003, Package_SO:TSSOP-16_4.4x5mm_P0.65mm, symbol Transistor_Array:ULN2003
Connections:
- net labels removed: +5V, CBUS0, CBUS1, CBUS2, CBUS3, LED_1_CTRL, LED_2_CTRL, LED_3_CTRL, RELAY_1_CTRL, RELAY_2_CTRL, RELAY_3_CTRL, RELAY_4_CTRL
- wire segments 98 -> 26
